File: temp_hum_board/temp_hum_board.kicad_sch (KiCad schematic)
At the start: 8 parts, among them SW1 SW_Push, SW2 SW_Push

Commit message: board temp hum
Parts:
- removed SW2: SW_Push, symbol Switch:SW_Push
- added BAT+, BAT-: TestPoint, symbol Connector:TestPoint
- added C? (x2): 2,2uF, symbol Device:C
- added R1: R, symbol Device:R
- added SW1: SW_Push, user_lib:tactile switch, symbol Switch:SW_Push
- added U1: CH340C, Package_SO:SOIC-16_3.9x9.9mm_P1.27mm, symbol Interface_USB:CH340C
- added U?: LD1117S33TR_SOT223, Package_TO_SOT_SMD:SOT-223-3_TabPin2, symbol Regulator_Linear:LD1117S33TR_SOT223
- C1: renamed from C2; value ?? -> 0,1µF; footprint (none) -> Capacitor_SMD:C_0402_1005Metric
- C2: renamed from C1; value ?? -> 0,1µF; footprint (none) -> Capacitor_SMD:C_0402_1005Metric
- P1: renamed from P?; footprint (none) -> Connector_USB:USB_C_Receptacle_HRO_TYPE-C-31-M-12
- R2: footprint (none) -> Resistor_SMD:R_0402_1005Metric
- R3: renamed from R1; footprint (none) -> Resistor_SMD:R_0402_1005Metric
- SW2: renamed from SW1; footprint (none) -> user_lib:tactile switch
- gave numbers to parts that had none: 1
Connections:
- net +3V3: now also C?.1, U?.2 (VO)
- net EN: now also SW1.1
- net GND: now also BAT-.1, C?.2, C?.2, R1.2, SW1.2, U1.1 (GND), U?.1 (GND)
- net VPP: now reaches P1.A4 (VBUS), P1.A9 (VBUS), P1.B4 (VBUS), P1.B9 (VBUS)
- net at P1.A5 (CC): now also R1.1
- net D+: now reaches P1.A6 (D+)
- net D+: now also P1.B6 (D+), U1.5 (UD+)
- net D-: now reaches P1.A7 (D-)
- net D-: now also P1.B7 (D-), U1.6 (UD-)
- net RXD0: now reaches U2.34 (RXD0)
- net RXD0: now also U1.2 (TXD)
- net TXD0: now reaches U2.35 (TXD0)
- net TXD0: now also U1.3 (RXD)
- new net +BATT: BAT+.1, C?.1, U?.3 (VI)
